File: ESP32_S3_MINI/ESP32-S3-MINI-1_UU.kicad_sch (KiCad schematic)
At the start: 50 parts, among them IC1 TPS6282533DMQR, IC2 BQ25185DLHR, J1 JST_2mm_LiPo, J2 USB4120-03-C, J3 Qwiic_Vertical, J4 Castellated_1x01, J5 Castellated_1x17, J6 Castellated_1x19, U2 ESP32-S3-MINI-1, U3 MAX17048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

Commit message: Design Review
Parts:
- added C13: 4.7uF, PCM_SparkFun-Capacitor:C_0402_1005Metric, symbol PCM_SparkFun-Capacitor:4.7uF_0402_6.3V_10%
- added C14: 10nF, PCM_SparkFun-Capacitor:C_0402_1005Metric, symbol PCM_SparkFun-Capacitor:10nF_0402_25V_10%
- added C15: 0.1uF, PCM_SparkFun-Capacitor:C_0402_1005Metric, symbol PCM_SparkFun-Capacitor:0.1uF_0402_16V_10%
- D7, D8: value ESD9B5.0ST5G -> ESD9101P2T5G
- R14, R16: value 2k2 -> 4k7
- R2: value 13k -> 18k
Connections:
- net 3V3: now also C13.2, C14.1
- net GND: now also J2.MH1, J2.MH2, J2.MH3, J2.MH4, C13.1, C14.2, C15.2
- net VBAT: now also C15.1
Other:
- note added: "Battery Monitor"
- note added: "Enable internal pull up for alert"
- note added: "R2 13k 1.1A 18k 0.5A 24k 0.1A"
- note removed: "Bettery Monitor"
- moved on the sheet: U3, U4
