File: ESP32_S3_MINI/ESP32-S3-MINI-1_UU.kicad_pcb (KiCad board)
At the start: 2 copper layers, 20.3 x 47 mm, 50 parts, among them IC1 TPS6282533DMQR, IC2 BQ25185DLHR, J1 JST_2mm_LiPo, J2 USB4120-03-C, J3 Qwiic_Vertical, J4 Castellated_1x01, J5 Castellated_1x17, J6 Castellated_1x19, U2 ESP32-S3-MINI-1, U3 MAX17048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

Commit message: Design Review
Parts:
- added C13: 4.7uF, PCM_SparkFun-Capacitor:C_0402_1005Metric, F.Cu at (205.5, 107.0)
- added C14: 10nF, PCM_SparkFun-Capacitor:C_0402_1005Metric, F.Cu at (203.2, 96.0)
- added C15: 0.1uF, PCM_SparkFun-Capacitor:C_0402_1005Metric, F.Cu at (200.1, 106.7)
- D7, D8: value ESD9B5.0ST5G -> ESD9101P2T5G
- R14, R16: value 2k2 -> 4k7
- R2: value 13k -> 18k
- moved C7 0.58 mm to (201.2, 105.0), turned to 90 degrees
Connections:
- J2 pad MH1: unconnected-(J2-PadMH1) -> GND
- J2 pad MH2: unconnected-(J2-PadMH2) -> GND
- J2 pad MH3: unconnected-(J2-PadMH3) -> GND
- J2 pad MH4: unconnected-(J2-PadMH4) -> GND
Routing:
- net GND: track 58.3 -> 67.9 mm
- net VBAT: track 14.3 -> 9.19 mm
- net 3V3: track 68.6 -> 69.8 mm

Commit message: Design Review
Other:
- board text added: "2026"
- board text added: "UU"
Changed lines of the file:
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@@
 		(layer "Edge.Cuts")
+	)
+	(gr_text "2026"
+		(at 206.8 113 0)
+		(layer "F.SilkS")
+		(effects
+			(font
+				(size 0.5 0.5)
+				(thickness 0.05)
+			)
+			(justify left bottom)
+		)
+	)
+	(gr_text "UU"
+		(at 206.6 114.3 0)
+		(layer "F.SilkS")
+		(effects
+			(font
+				(size 1 1)
+				(thickness 0.1)
+			)
+			(justify left bottom)
+		)
+	)
+	(gr_text "2026"
+		(at 208.7 113 0)
+		(layer "B.SilkS")
+		(effects
+			(font
+				(size 0.5 0.5)
+				(thickness 0.05)
+			)
+			(justify left bottom mirror)
+		)
+	)
+	(gr_text "UU"
+		(at 208.8 114.3 0)
+		(layer "B.SilkS")
+		(effects
+			(font
+				(size 1 1)
+				(thickness 0.1)
+			)
+			(justify left bottom mirror)
+		)
 	)
 	(dimension

Commit message: BOM
Other:
- board text added: "10"
- board text added: "11"
- board text added: "12"
- board text added: "13"
- board text added: "14"
- board text added: "15"
- board text added: "16"
- board text added: "17"
- board text added: "18"
- board text added: "2"
- board text added: "21"
- board text added: "26"
- board text added: "3"
- board text added: "33"
- board text added: "34"
- board text added: "35"
- board text added: "36"
- board text added: "37"
- board text added: "38"
- board text added: "3V3"
- board text added: "4"
- board text added: "46"
- board text added: "47"
- board text added: "5"
- board text added: "6"
- board text added: "7"
- board text added: "BAT"
- board text added: "BAT_CHRG"
- board text added: "BOOT"
- board text added: "CHRG"
- board text added: "ESP32 S3 MINI"
- board text added: "GND"
- board text added: "LED"
- board text added: "MTCK"
- board text added: "MTDI"
- board text added: "MTDO"
- board text added: "MTMS"
- board text added: "RESET"
- board text added: "RGB"
- board text added: "RX"
- board text added: "TEMP"
- board text added: "TX"
- board text added: "USB 2.0"
- board text added: "V_REG"
- board text added: "V_USB"

Commit message: Cleanup
Routing:
- net GND: track 67.9 -> 71.0 mm, vias 33 -> 37

Commit message: Labels
Other:
- board text added: "45"
